Commit message: 3 korrigieren

File: catkin_ws/src/mbot_description/urdf/mbot_base.xacro (robot description, xacro)
@@ -68,5 +68,5 @@
             </visual>
         </link>
-        <joint name="base_footprint_joint" type="fixed"><!-- 让机器人的base_link上移，至车轮与水平线平齐 -->
+        <joint name="base_footprint_joint" type="fixed">
             <origin xyz="0 0 ${base_length/2 + caster_radius*2}" rpy="0 0 0" />
             <parent link="base_footprint"/>
@@ -83,7 +83,7 @@
         </link>
     </xacro:macro>
-        <xacro:wheel prefix="left" reflect="-1"/> <!-- 调用驱动轮子宏定义 -->
-        <xacro:wheel prefix="right" reflect="1"/> <!-- 调用驱动轮子宏定义 -->
-        <xacro:caster prefix="front" reflect="-1"/> <!-- 调用支撑轮子宏定义 -->
-        <xacro:caster prefix="back" reflect="1"/> <!-- 调用支撑轮子宏定义 -->
+        <xacro:wheel prefix="left" reflect="-1"/>
+        <xacro:wheel prefix="right" reflect="1"/>
+        <xacro:caster prefix="front" reflect="-1"/>
+        <xacro:caster prefix="back" reflect="1"/>
 </robot>
