Commit message: 08.07 first

File: catkin_ws/src/mbot_description/urdf/mbot.gazebo.xacro (robot description, xacro)
@@ -15,9 +15,48 @@
   <!--caster-->
   <gazebo reference="caster">
+    <mu1>0.2</mu1>
+    <mu2>0.2</mu2>
     <material>Gazebo/Black</material>
   </gazebo>
   <!--wheel-->
   <gazebo reference="wheel">
+    <mu1>0.2</mu1>
+    <mu2>0.2</mu2>
     <material>Gazebo/Gray</material>
   </gazebo>
+    <!--camera_link-->
+  <gazebo reference="camera_model">
+    <material>Gazebo/Grey</material>
+  </gazebo>
+  <!-- camera-->
+  <gazebo reference="camera_link">
+    <sensor type="camera" name="rgb_camera">
+      <update_rate>30.0</update_rate>
+      <camera name="rgb_camera">
+        <horizontal_fov>1.4</horizontal_fov>
+        <image>
+          <width>640</width>
+          <height>480</height>
+          <format>R8G8B8</format>
+        </image>
+        <clip>
+          <near>0.02</near>
+          <far>300</far>
+        </clip>
+      </camera>
+      <plugin name="camera_controller" filename="libgazebo_ros_camera.so">
+        <alwaysOn>true</alwaysOn>
+        <updateRate>0.0</updateRate>
+        <imageTopicName>image_raw</imageTopicName>
+        <cameraInfoTopicName>camera_info</cameraInfoTopicName>
+        <frameName>camera_link</frameName>
+        <hackBaseline>0.0</hackBaseline>
+        <distortionK1>0.0</distortionK1>
+        <distortionK2>0.0</distortionK2>
+        <distortionK3>0.0</distortionK3>
+        <distortionT1>0.0</distortionT1>
+        <distortionT2>0.0</distortionT2>
+      </plugin>
+    </sensor>
+  </gazebo>
 </robot>

File: catkin_ws/src/mbot_description/urdf/mbot_base.xacro (robot description, xacro)
@@ -14,4 +14,5 @@
     <xacro:property name="caster_joint_x" value="0.18"/>
     <xacro:include filename="materials.xacro" />
+    <!-- Macro for inertia matrix-->
     <xacro:macro name="sphere_inertial_matrix" params="m r">
         <inertial>
@@ -30,6 +31,13 @@
         </inertial>
     </xacro:macro>
+    <xacro:macro name="box_inertial_matrix" params="m w h d">
+        <inertial>
+            <mass value="${m}" />
+            <inertia ixx="${m*(h*h+d*d)/12}" ixy = "0" ixz = "0"
+                iyy="${m*(w*w+d*d)/12}" iyz = "0"
+                izz="${m*(w*w+h*h)/12}" />
+        </inertial>
+    </xacro:macro>
     <!--classis motorwheel-->
-    <!--prefix（left or right） reflect（mirror relationship）-->
     <xacro:macro name="wheel" params="prefix reflect">
         <joint name="${prefix}_wheel_joint" type="continuous">
@@ -53,9 +61,10 @@
                 </geometry>
             </collision>
-            <cylinder_inertial_matrix  m="${wheel_mass}" r="${wheel_radius}" h="${wheel_length}" />
+            <xacro:cylinder_inertial_matrix  m="${wheel_mass}" r="${wheel_radius}" h="${wheel_length}" />
         </link>
         <gazebo reference="${prefix}_wheel_link">
             <material>Gazebo/Gray</material>
         </gazebo>
+        <!-- Transmission is important to link the joints and the controller -->
         <transmission name="${prefix}_wheel_joint_trans">
             <type>transmission_interface/SimpleTransmission</type>
@@ -91,5 +100,5 @@
                 </geometry>
             </collision>
-            <sphere_inertial_matrix  m="${caster_mass}" r="${caster_radius}" />
+            <xacro:sphere_inertial_matrix  m="${caster_mass}" r="${caster_radius}" />
         </link>
         <gazebo reference="${prefix}_caster_link">
@@ -129,5 +138,5 @@
                 </geometry>
             </collision>
-            <cylinder_inertial_matrix  m="${base_mass}" r="${base_radius}" h="${base_length}" />
+            <xacro:cylinder_inertial_matrix  m="${base_mass}" r="${base_radius}" h="${base_length}" />
         </link>
         <gazebo reference="base_link">
@@ -139,7 +148,9 @@
         <xacro:caster prefix="front" reflect="-1"/>
         <xacro:caster prefix="back" reflect="1"/>
+	<!-- controller -->
         <gazebo>
             <plugin name="differential_drive_controller"
                     filename="libgazebo_ros_diff_drive.so">
+		<alwaysOn>true</alwaysOn>
                 <rosDebugLevel>Debug</rosDebugLevel>
                 <publishWheelTF>true</publishWheelTF>
@@ -161,4 +172,6 @@
                 <odometryTopic>odom</odometryTopic>
                 <robotBaseFrame>base_footprint</robotBaseFrame>
+                <publishOdomTF>true</publishOdomTF>
+                <odometrySource> 1</odometrySource>
             </plugin>
         </gazebo>
