Commit message: before reinstall ubuntu 18

File: copy.xacro (robot description, xacro)
@@ -11,7 +11,15 @@
     <xacro:property name="wheel_joint_z" value="0.05"/>
     <xacro:property name="caster_mass"    value="0.5" />
-    <xacro:property name="caster_radius" value="0.015"/>
+    <xacro:property name="caster_radius"  value="0.015"/>
     <xacro:property name="caster_joint_x" value="0.18"/>
-    <xacro:include filename="materials.xacro" />
+    <material name="yellow">
+        <color rgba="1 0.4 0 1"/>
+    </material>
+    <material name="black">
+        <color rgba="0 0 0 0.95"/>
+    </material>
+    <material name="gray">
+        <color rgba="0.75 0.75 0.75 1"/>
+    </material>
     <xacro:macro name="sphere_inertial_matrix" params="m r">
         <inertial>
@@ -30,6 +38,4 @@
         </inertial>
     </xacro:macro>
-    <!--classis motorwheel-->
-    <!--prefix（left or right） reflect（mirror relationship）-->
     <xacro:macro name="wheel" params="prefix reflect">
         <joint name="${prefix}_wheel_joint" type="continuous">
@@ -69,6 +75,5 @@
         </transmission>
     </xacro:macro>
-   <!--caster-->
-     <xacro:macro name="caster" params="prefix reflect">
+    <xacro:macro name="caster" params="prefix reflect">
         <joint name="${prefix}_caster_joint" type="continuous">
             <origin xyz="${reflect*caster_joint_x} 0 ${-(base_length/2 + caster_radius)}" rpy="0 0 0"/>
@@ -97,6 +102,5 @@
         </gazebo>
     </xacro:macro>
-    <!--base_footprint -->
-        <xacro:macro name="mbot_base">
+    <xacro:macro name="mbot_base_gazebo">
         <link name="base_footprint">
             <visual>
@@ -134,9 +138,9 @@
             <material>Gazebo/Blue</material>
         </gazebo>
+        <wheel prefix="left" reflect="-1"/>
+        <wheel prefix="right" reflect="1"/>
+        <caster prefix="front" reflect="-1"/>
+        <caster prefix="back" reflect="1"/>
     </xacro:macro>
-        <xacro:wheel prefix="left" reflect="-1"/>
-        <xacro:wheel prefix="right" reflect="1"/>
-        <xacro:caster prefix="front" reflect="-1"/>
-        <xacro:caster prefix="back" reflect="1"/>
         <gazebo>
             <plugin name="differential_drive_controller"
